File: PCB Diagrams/IR-Keyboard-Mouse-Emulator.kicad_pcb (KiCad board)
At the start: 2 copper layers, 22.9 x 43.2 mm, 4 parts, among them U1 VS1838B, U2 ProMicroC

Commit message: update schematics and pcb
Parts:
- R1: footprint Resistor_THT:R_Axial_DIN0204_L3.6mm_D1.6mm_P5.08mm_Horizontal -> Resistor_THT:R_Axial_DIN0207_L6.3mm_D2.5mm_P7.62mm_Horizontal
- moved R1 7.62 mm to (154.9, 101.6), turned to -90 degrees
Connections:
- D1 pad 1: GND -> Net-(D1-K)
- R1 pad 1: Net-(D1-A) -> Net-(U2-D14)
- R1 pad 2: Net-(U2-D14) -> Net-(D1-A)
- U1 pad 1: (no net) -> Net-(U1-OUT)
- U1 pad 2: (no net) -> Net-(D1-K)
- U1 pad 3: (no net) -> +5V
- U2 pad 23: GND -> Net-(D1-K)
- U2 pad 4: GND -> Net-(D1-K)
Routing:
- net Net-(D1-K): track 0.00 -> 55.5 mm
- net GND: track 39.7 -> 0.00 mm
- net Net-(U2-D14): track 5.08 -> 6.13 mm
Changed lines of the file:
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@@
 	)
 	(net 0 "")
-	(net 1 "GND")
+	(net 1 "Net-(D1-K)")
 	(net 2 "Net-(D1-A)")
 	(net 3 "Net-(U1-OUT)")
@@
 		)
 		(sheetname "/")
-		(sheetfile "IR-Keyboard-Mouse-Emulator-KiCAD.kicad_sch")
+		(sheetfile "IR-Keyboard-Mouse-Emulator.kicad_sch")
 		(fp_line
 			(start -8.89 -16.51)
@@
 			(remove_unused_layers no)
 			(roundrect_rratio 0.5)
-			(net 1 "GND")
+			(net 1 "Net-(D1-K)")
 			(pinfunction "GND")
-			(pintype "input")
+			(pintype "passive")
 			(thermal_bridge_angle 0)
 		)
@@
 			(net 4 "+5V")
 			(pinfunction "5V")
-			(pintype "input")
+			(pintype "power_in")
 			(thermal_bridge_angle 0)
 		)
@@
 			(remove_unused_layers no)
 			(roundrect_rratio 0.5)
-			(net 1 "GND")
+			(net 1 "Net-(D1-K)")
 			(pinfunction "GND")
-			(pintype "input")
+			(pintype "passive")
 			(thermal_bridge_angle 0)
 		)
@@
 	(footprint "OptoDevice:Vishay_MINICAST-3Pin"
 		(layer "F.Cu")
-		(at 144.78 113.04)
+		(at 144.78 113.03)
 		(descr "IR Receiver Vishay TSOP-xxxx, MINICAST package, see https://www.vishay.com/docs/82669/tsop32s40f.pdf")
 		(tags "IR Receiver Vishay TSOP-xxxx MINICAST")
 		(property "Reference" "U1"
-			(at -2.54 0 0)
+			(at -2.2 1.27 180)
 			(layer "F.SilkS")
 			(effects
@@
 		)
 		(property "Value" "VS1838B"
-			(at 2.54 2.54 0)
+			(at 2.54 2.54 180)
 			(layer "F.Fab")
 			(effects
 				(font
 					(size 1 1)
-					(thickness 0.15)
-				)
-			)
-		)
-		(property "Datasheet" "Datasheet not available"
+					(thickness 0.12)
+				)
+			)
+		)
+		(property "Datasheet" ""
 			(at 0 0 0)
 			(unlocked yes)
@@
 			)
 		)
+		(property ki_fp_filters "Vishay*CAST*")
+		(sheetname "/")
+		(sheetfile "IR-Keyboard-Mouse-Emulator.kicad_sch")
 		(attr through_hole)
 		(fp_line
@@
 			(at 0 0)
 			(size 1.8 1.8)
-			(drill 0.9)
+			(drill 1)
 			(layers "*.Cu" "*.Mask")
 			(remove_unused_layers no)
 			(roundrect_rratio 0.139)
+			(net 3 "Net-(U1-OUT)")
 			(pinfunction "OUT")
 			(pintype "output")
@@
 			(at 2.54 0)
 			(size 1.8 1.8)
-			(drill 0.9)
-			(layers "*.Cu" "*.Mask")
-			(remove_unused_layers no)
+			(drill 1)
+			(layers "*.Cu" "*.Mask")
+			(remove_unused_layers no)
+			(net 1 "Net-(D1-K)")
 			(pinfunction "GND")
-			(pintype "power_in")
+			(pintype "passive")
 		)
 		(pad "3" thru_hole circle
 			(at 5.08 0)
 			(size 1.8 1.8)
-			(drill 0.9)
-			(layers "*.Cu" "*.Mask")
-			(remove_unused_layers no)
+			(drill 1)
+			(layers "*.Cu" "*.Mask")
+			(remove_unused_layers no)
+			(net 4 "+5V")
 			(pinfunction "VSS")
 			(pintype "power_in")
@@
 			(at 1.27 0 0)
 			(layer "F.Fab")
+			(hide yes)
 			(effects
 				(font
@@
 		(property ki_fp_filters "LED* LED_SMD:* LED_THT:*")
 		(sheetname "/")
-		(sheetfile "IR-Keyboard-Mouse-Emulator-KiCAD.kicad_sch")
+		(sheetfile "IR-Keyboard-Mouse-Emulator.kicad_sch")
 		(attr through_hole)
 		(fp_line
@@
 			(at 0 0 90)
 			(size 1.8 1.8)
-			(drill 0.9)
-			(layers "*.Cu" "*.Mask")
-			(remove_unused_layers no)
-			(net 1 "GND")
+			(drill 1)
+			(layers "*.Cu" "*.Mask")
+			(remove_unused_layers no)
+			(net 1 "Net-(D1-K)")
 			(pinfunction "K")
 			(pintype "passive")
@@
 			(at 2.54 0 90)
 			(size 1.8 1.8)
-			(drill 0.9)
+			(drill 1)
 			(layers "*.Cu" "*.Mask")
 			(remove_unused_layers no)
@@
 		)
 	)
-	(footprint "Resistor_THT:R_Axial_DIN0204_L3.6mm_D1.6mm_P5.08mm_Horizontal"
+	(footprint "Resistor_THT:R_Axial_DIN0207_L6.3mm_D2.5mm_P7.62mm_Horizontal"
 		(layer "F.Cu")
-		(at 154.94 109.22 90)
-		(descr "Resistor, Axial_DIN0204 series, Axial, Horizontal, pin pitch=5.08mm, 0.167W, length*diameter=3.6*1.6mm^2, http://cdn-reichelt.de/documents/datenblatt/B400/1_4W%23YAG.pdf")
-		(tags "Resistor Axial_DIN0204 series Axial Horizontal pin pitch 5.08mm 0.167W length 3.6mm diameter 1.6mm")
+		(at 154.94 101.6 -90)
+		(descr "Resistor, Axial_DIN0207 series, Axial, Horizontal, pin pitch=7.62mm, 0.25W = 1/4W, length*diameter=6.3*2.5mm^2, http://cdn-reichelt.de/documents/datenblatt/B400/1_4W%23YAG.pdf")
+		(tags "Resistor Axial_DIN0207 series Axial Horizontal pin pitch 7.62mm 0.25W = 1/4W length 6.3mm diameter 2.5mm")
 		(property "Reference" "R1"
-			(at 2.54 -2.54 90)
+			(at 3.81 2.54 180)
 			(layer "F.SilkS")
 			(effects
@@
 		)
 		(property "Value" "1K"
-			(at 2.54 0 90)
+			(at 3.81 0 90)
 			(layer "F.Fab")
 			(effects
@@
 		(property ki_fp_filters "R_*")
 		(sheetname "/")
-		(sheetfile "IR-Keyboard-Mouse-Emulator-KiCAD.kicad_sch")
+		(sheetfile "IR-Keyboard-Mouse-Emulator.kicad_sch")
 		(attr through_hole)
 		(fp_line
-			(start 0.62 -0.92)
-			(end 4.46 -0.92)
-			(stroke
-				(width 0.12)
-				(type solid)
-			)
-			(layer "F.SilkS")
-		)
-		(fp_line
-			(start 0.62 0.92)
-			(end 4.46 0.92)
+			(start 0.54 1.37)
+			(end 7.08 1.37)
+			(stroke
+				(width 0.12)
+				(type solid)
+			)
+			(layer "F.SilkS")
+		)
+		(fp_line
+			(start 7.08 1.37)
+			(end 7.08 1.04)
+			(stroke
+				(width 0.12)
+				(type solid)
+			)
+			(layer "F.SilkS")
+		)
+		(fp_line
+			(start 0.54 1.04)
+			(end 0.54 1.37)
+			(stroke
+				(width 0.12)
+				(type solid)
+			)
+			(layer "F.SilkS")
+		)
+		(fp_line
+			(start 0.54 -1.04)
+			(end 0.54 -1.37)
+			(stroke
+				(width 0.12)
+				(type solid)
+			)
+			(layer "F.SilkS")
+		)
+		(fp_line
+			(start 0.54 -1.37)
+			(end 7.08 -1.37)
+			(stroke
+				(width 0.12)
+				(type solid)
+			)
+			(layer "F.SilkS")
+		)
+		(fp_line
+			(start 7.08 -1.37)
+			(end 7.08 -1.04)
 			(stroke
 				(width 0.12)
@@
 		)
 		(fp_rect
-			(start -0.95 -1.05)
-			(end 6.03 1.05)
+			(start -1.05 -1.5)
+			(end 8.67 1.5)
 			(stroke
 				(width 0.05)
@@
 		)
 		(fp_line
-			(start 5.08 0)
-			(end 4.34 0)
+			(start 0 0)
+			(end 0.66 0)
 			(stroke
 				(width 0.1)
@@
 		)
 		(fp_line
-			(start 0 0)
-			(end 0.74 0)
+			(start 7.62 0)
+			(end 6.96 0)
 			(stroke
 				(width 0.1)
@@
 		)
 		(fp_rect
-			(start 0.74 -0.8)
-			(end 4.34 0.8)
+			(start 0.66 -1.25)
+			(end 6.96 1.25)
 			(stroke
 				(width 0.1)
@@
 		)
 		(pad "1" thru_hole circle
-			(at 0 0 90)
-			(size 1.4 1.4)
-			(drill 0.7)
+			(at 0 0 270)
+			(size 1.6 1.6)
+			(drill 0.8)
+			(layers "*.Cu" "*.Mask")
+			(remove_unused_layers no)
+			(net 11 "Net-(U2-D14)")
+			(pintype "passive")
+		)
+		(pad "2" thru_hole circle
+			(at 7.62 0 270)
+			(size 1.6 1.6)
+			(drill 0.8)
 			(layers "*.Cu" "*.Mask")
 			(remove_unused_layers no)
@@
 			(pintype "passive")
 		)
-		(pad "2" thru_hole circle
-			(at 5.08 0 90)
-			(size 1.4 1.4)
-			(drill 0.7)
-			(layers "*.Cu" "*.Mask")
-			(remove_unused_layers no)
-			(net 11 "Net-(U2-D14)")
-			(pintype "passive")
-		)
 		(embedded_fonts no)
-		(model "${KICAD9_3DMODEL_DIR}/Resistor_THT.3dshapes/R_Axial_DIN0204_L3.6mm_D1.6mm_P5.08mm_Horizontal.step"
+		(model "${KICAD9_3DMODEL_DIR}/Resistor_THT.3dshapes/R_Axial_DIN0207_L6.3mm_D2.5mm_P7.62mm_Horizontal.step"
 			(offset
 				(xyz 0 0 0)
@@
 	)
 	(segment
+		(start 147.32 91.44)
+		(end 154.94 83.82)
+		(width 1)
+		(layer "B.Cu")
+		(net 1)
+	)
+	(segment
 		(start 147.32 113.03)
 		(end 147.32 91.44)
@@
 	)
 	(segment
+		(start 154.94 83.82)
+		(end 160.02 83.82)
+		(width 1)
+		(layer "B.Cu")
+		(net 1)
+	)
+	(segment
 		(start 148.59 115.57)
 		(end 147.32 114.3)
@@
 	)
 	(segment
-		(start 154.94 104.14)
+		(start 157.48 101.6)
 		(end 160.02 104.14)
 		(width 1)
 		(layer "B.Cu")
+		(net 11)
+	)
+	(segment
+		(start 154.94 101.6)
+		(end 157.48 101.6)
+		(width 1)
+		(layer "B.Cu")
