File: PCB Diagrams/Version Allways On/IR-Keyboard-Mouse-Emulator.kicad_pcb (KiCad board)
At the start: 2 copper layers, 22.9 x 43.2 mm, 4 parts, among them U1 VS1838B, U2 ProMicroC

Commit message: Adding Low Power protoboard & schematics diagram
Parts:
- R1: value 1K -> 10K
- U2: value ProMicroC -> Arduino_Pro_Micro
Changed lines of the file:
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@@
 		(tags "SparkFun")
 		(property "Reference" "U2"
-			(at 0 0 0)
+			(at 0 -13.97 180)
 			(layer "F.Fab")
 			(effects
@@
 			)
 		)
-		(property "Value" "ProMicroC"
-			(at 0 -5.08 0)
+		(property "Value" "Arduino_Pro_Micro"
+			(at 0 0 90)
 			(layer "F.Fab")
 			(effects
@@
 		(tags "IR Receiver Vishay TSOP-xxxx MINICAST")
 		(property "Reference" "U1"
-			(at -2.2 1.27 180)
+			(at -2.3 0 180)
 			(layer "F.SilkS")
 			(effects
@@
 			)
 		)
-		(property "Value" "1K"
+		(property "Value" "10K"
 			(at 3.81 0 90)
 			(layer "F.Fab")

Commit message: Adding Low Power protoboard & schematics diagram
Parts:
- R1: footprint Resistor_THT:R_Axial_DIN0207_L6.3mm_D2.5mm_P7.62mm_Horizontal -> Resistor_THT:R_Axial_DIN0204_L3.6mm_D1.6mm_P5.08mm_Horizontal
- U2: footprint PCM_SparkFun-Board:ProMicroC -> Custom:Arduino_Pro_Micro
- moved R1 2.54 mm to (154.9, 104.1)
Routing:
- net Net-(U2-D14): track 6.13 -> 5.08 mm
