File: PCB Diagrams/Version Allways On/IR-Keyboard-Mouse-Emulator.kicad_sch (KiCad schematic)
At the start: 4 parts, among them U1 VS1838B, U2 ProMicroC

Commit message: Adding Low Power protoboard & schematics diagram
Parts:
- R1: value 1K -> 10K
- U2: value ProMicroC -> Arduino_Pro_Micro
Changed lines of the file:
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@@
 			)
 		)
-		(property "Value" "ProMicroC"
+		(property "Value" "Arduino_Pro_Micro"
 			(at 152.146 82.296 0)
 			(effects
@@
 			)
 		)
-		(property "Value" "1K"
+		(property "Value" "10K"
 			(at 167.64 102.87 90)
 			(effects

Commit message: Adding Low Power protoboard & schematics diagram
Parts:
- R1: footprint Resistor_THT:R_Axial_DIN0207_L6.3mm_D2.5mm_P7.62mm_Horizontal -> Resistor_THT:R_Axial_DIN0204_L3.6mm_D1.6mm_P5.08mm_Horizontal
- U2: footprint PCM_SparkFun-Board:ProMicroC -> Custom:Arduino_Pro_Micro
Changed lines of the file:
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@@
 			)
 		)
-		(property "Footprint" "PCM_SparkFun-Board:ProMicroC"
+		(property "Footprint" "Custom:Arduino_Pro_Micro"
 			(at 147.574 122.936 0)
 			(effects
@@
 			)
 		)
-		(property "Footprint" "Resistor_THT:R_Axial_DIN0207_L6.3mm_D2.5mm_P7.62mm_Horizontal"
+		(property "Footprint" "Resistor_THT:R_Axial_DIN0204_L3.6mm_D1.6mm_P5.08mm_Horizontal"
 			(at 165.862 102.87 90)
 			(effects
